File: Hardware/Schematics/LoRa RF.kicad_sch (KiCad schematic)
At the start: 17 parts, among them J6 Conn_Coaxial, U4 BGS12WN6E6327

Commit message: title block update
Other:
- company: (none) -> Nicola Borkowetz
- title: (none) -> LoRa Node RF
Changed lines of the file:
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@@
 	(generator_version "10.0")
 	(paper "A4")
+	(title_block
+		(title "LoRa Node RF")
+		(date "2025-11-28")
+		(rev "A")
+		(company "Nicola Borkowetz")
+	)
 	(junction
 		(at 59.69 67.31)
@@
 		)
 		(instances
-			(project "demo wateranalyser"
+			(project "demo LoRa_Node"
 				(path "/3e989608-eeda-4a48-bc6c-c5e1d1678702/f7bd652a-238e-4a19-a7e7-e5372eb58a34"
 					(reference "C21")
@@
 		)
 		(instances
-			(project "demo wateranalyser"
+			(project "demo LoRa_Node"
 				(path "/3e989608-eeda-4a48-bc6c-c5e1d1678702/f7bd652a-238e-4a19-a7e7-e5372eb58a34"
 					(reference "#PWR046")
@@
 		)
 		(instances
-			(project "demo wateranalyser"
+			(project "demo LoRa_Node"
 				(path "/3e989608-eeda-4a48-bc6c-c5e1d1678702/f7bd652a-238e-4a19-a7e7-e5372eb58a34"
 					(reference "L2")
@@
 		)
 		(instances
-			(project "demo wateranalyser"
+			(project "demo LoRa_Node"
 				(path "/3e989608-eeda-4a48-bc6c-c5e1d1678702/f7bd652a-238e-4a19-a7e7-e5372eb58a34"
 					(reference "C26")
@@
 		)
 		(instances
-			(project "demo wateranalyser"
+			(project "demo LoRa_Node"
 				(path "/3e989608-eeda-4a48-bc6c-c5e1d1678702/f7bd652a-238e-4a19-a7e7-e5372eb58a34"
 					(reference "#PWR045")
@@
 		)
 		(instances
-			(project "demo wateranalyser"
+			(project "demo LoRa_Node"
 				(path "/3e989608-eeda-4a48-bc6c-c5e1d1678702/f7bd652a-238e-4a19-a7e7-e5372eb58a34"
 					(reference "#PWR041")
@@
 		)
 		(instances
-			(project "demo wateranalyser"
+			(project "demo LoRa_Node"
 				(path "/3e989608-eeda-4a48-bc6c-c5e1d1678702/f7bd652a-238e-4a19-a7e7-e5372eb58a34"
 					(reference "C23")
@@
 		)
 		(instances
-			(project "demo wateranalyser"
+			(project "demo LoRa_Node"
 				(path "/3e989608-eeda-4a48-bc6c-c5e1d1678702/f7bd652a-238e-4a19-a7e7-e5372eb58a34"
 					(reference "#PWR038")
@@
 		)
 		(instances
-			(project "demo wateranalyser"
+			(project "demo LoRa_Node"
 				(path "/3e989608-eeda-4a48-bc6c-c5e1d1678702/f7bd652a-238e-4a19-a7e7-e5372eb58a34"
 					(reference "C28")
@@
 		)
 		(instances
-			(project "demo wateranalyser"
+			(project "demo LoRa_Node"
 				(path "/3e989608-eeda-4a48-bc6c-c5e1d1678702/f7bd652a-238e-4a19-a7e7-e5372eb58a34"
 					(reference "J6")
@@
 		)
 		(instances
-			(project "demo wateranalyser"
+			(project "demo LoRa_Node"
 				(path "/3e989608-eeda-4a48-bc6c-c5e1d1678702/f7bd652a-238e-4a19-a7e7-e5372eb58a34"
 					(reference "U4")
@@
 		)
 		(instances
-			(project "demo wateranalyser"
+			(project "demo LoRa_Node"
 				(path "/3e989608-eeda-4a48-bc6c-c5e1d1678702/f7bd652a-238e-4a19-a7e7-e5372eb58a34"
 					(reference "C22")
@@
 		)
 		(instances
-			(project "demo wateranalyser"
+			(project "demo LoRa_Node"
 				(path "/3e989608-eeda-4a48-bc6c-c5e1d1678702/f7bd652a-238e-4a19-a7e7-e5372eb58a34"
 					(reference "C25")
@@
 		)
 		(instances
-			(project "demo wateranalyser"
+			(project "demo LoRa_Node"
 				(path "/3e989608-eeda-4a48-bc6c-c5e1d1678702/f7bd652a-238e-4a19-a7e7-e5372eb58a34"
 					(reference "#PWR039")
@@
 		)
 		(instances
-			(project "demo wateranalyser"
+			(project "demo LoRa_Node"
 				(path "/3e989608-eeda-4a48-bc6c-c5e1d1678702/f7bd652a-238e-4a19-a7e7-e5372eb58a34"
 					(reference "#PWR043")
@@
 		)
 		(instances
-			(project "demo wateranalyser"
+			(project "demo LoRa_Node"
 				(path "/3e989608-eeda-4a48-bc6c-c5e1d1678702/f7bd652a-238e-4a19-a7e7-e5372eb58a34"
 					(reference "#PWR040")
@@
 		)
 		(instances
-			(project "demo wateranalyser"
+			(project "demo LoRa_Node"
 				(path "/3e989608-eeda-4a48-bc6c-c5e1d1678702/f7bd652a-238e-4a19-a7e7-e5372eb58a34"
 					(reference "#PWR044")
@@
 		)
 		(instances
-			(project "demo wateranalyser"
+			(project "demo LoRa_Node"
 				(path "/3e989608-eeda-4a48-bc6c-c5e1d1678702/f7bd652a-238e-4a19-a7e7-e5372eb58a34"
 					(reference "L3")
@@
 		)
 		(instances
-			(project "demo wateranalyser"
+			(project "demo LoRa_Node"
 				(path "/3e989608-eeda-4a48-bc6c-c5e1d1678702/f7bd652a-238e-4a19-a7e7-e5372eb58a34"
 					(reference "C24")
@@
 		)
 		(instances
-			(project "demo wateranalyser"
+			(project "demo LoRa_Node"
 				(path "/3e989608-eeda-4a48-bc6c-c5e1d1678702/f7bd652a-238e-4a19-a7e7-e5372eb58a34"
 					(reference "C29")
@@
 		)
 		(instances
-			(project "demo wateranalyser"
+			(project "demo LoRa_Node"
 				(path "/3e989608-eeda-4a48-bc6c-c5e1d1678702/f7bd652a-238e-4a19-a7e7-e5372eb58a34"
 					(reference "L6")
@@
 		)
 		(instances
-			(project "demo wateranalyser"
+			(project "demo LoRa_Node"
 				(path "/3e989608-eeda-4a48-bc6c-c5e1d1678702/f7bd652a-238e-4a19-a7e7-e5372eb58a34"
 					(reference "#PWR042")
@@
 		)
 		(instances
-			(project "demo wateranalyser"
+			(project "demo LoRa_Node"
 				(path "/3e989608-eeda-4a48-bc6c-c5e1d1678702/f7bd652a-238e-4a19-a7e7-e5372eb58a34"
 					(reference "L4")
@@
 		)
 		(instances
-			(project "demo wateranalyser"
+			(project "demo LoRa_Node"
 				(path "/3e989608-eeda-4a48-bc6c-c5e1d1678702/f7bd652a-238e-4a19-a7e7-e5372eb58a34"
 					(reference "#PWR037")
@@
 		)
 		(instances
-			(project "demo wateranalyser"
+			(project "demo LoRa_Node"
 				(path "/3e989608-eeda-4a48-bc6c-c5e1d1678702/f7bd652a-238e-4a19-a7e7-e5372eb58a34"
 					(reference "L5")
@@
 		)
 		(instances
-			(project "demo wateranalyser"
+			(project "demo LoRa_Node"
 				(path "/3e989608-eeda-4a48-bc6c-c5e1d1678702/f7bd652a-238e-4a19-a7e7-e5372eb58a34"
 					(reference "C30")
@@
 		)
 		(instances
-			(project "demo wateranalyser"
+			(project "demo LoRa_Node"
 				(path "/3e989608-eeda-4a48-bc6c-c5e1d1678702/f7bd652a-238e-4a19-a7e7-e5372eb58a34"
 					(reference "C27")

Commit message: adjustment to the power section
Parts:
- renumbered C21 to C20, C22 to C21, C23 to C22, C24 to C23, C25 to C24, C26 to C25, C27 to C26, C28 to C27, C29 to C28, C30 to C29
Changed lines of the file:
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@@
 		(in_pos_files yes)
 		(dnp no)
-		(property "Reference" "C21"
+		(property "Reference" "C20"
 			(at 46.99 52.0699 0)
 			(show_name no)
@@
 			(project "demo LoRa_Node"
 				(path "/3e989608-eeda-4a48-bc6c-c5e1d1678702/f7bd652a-238e-4a19-a7e7-e5372eb58a34"
-					(reference "C21")
+					(reference "C20")
 					(unit 1)
 				)
@@
 		(in_pos_files yes)
 		(dnp no)
-		(property "Reference" "#PWR046"
+		(property "Reference" "#PWR045"
 			(at 85.09 162.56 0)
 			(hide yes)
@@
 			(project "demo LoRa_Node"
 				(path "/3e989608-eeda-4a48-bc6c-c5e1d1678702/f7bd652a-238e-4a19-a7e7-e5372eb58a34"
-					(reference "#PWR046")
+					(reference "#PWR045")
 					(unit 1)
 				)
@@
 		(in_pos_files yes)
 		(dnp no)
-		(property "Reference" "C26"
+		(property "Reference" "C25"
 			(at 210.82 81.28 90)
 			(show_name no)
@@
 			(project "demo LoRa_Node"
 				(path "/3e989608-eeda-4a48-bc6c-c5e1d1678702/f7bd652a-238e-4a19-a7e7-e5372eb58a34"
-					(reference "C26")
+					(reference "C25")
 					(unit 1)
 				)
@@
 		(in_pos_files yes)
 		(dnp no)
-		(property "Reference" "#PWR045"
+		(property "Reference" "#PWR044"
 			(at 240.03 113.03 0)
 			(hide yes)
@@
 			(project "demo LoRa_Node"
 				(path "/3e989608-eeda-4a48-bc6c-c5e1d1678702/f7bd652a-238e-4a19-a7e7-e5372eb58a34"
-					(reference "#PWR045")
+					(reference "#PWR044")
 					(unit 1)
 				)
@@
 		(in_pos_files yes)
 		(dnp no)
-		(property "Reference" "#PWR041"
+		(property "Reference" "#PWR040"
 			(at 129.54 90.17 0)
 			(hide yes)
@@
 			(project "demo LoRa_Node"
 				(path "/3e989608-eeda-4a48-bc6c-c5e1d1678702/f7bd652a-238e-4a19-a7e7-e5372eb58a34"
-					(reference "#PWR041")
+					(reference "#PWR040")
 					(unit 1)
 				)
@@
 		(in_pos_files yes)
 		(dnp no)
-		(property "Reference" "C23"
+		(property "Reference" "C22"
 			(at 109.22 60.96 90)
 			(show_name no)
@@
 			(project "demo LoRa_Node"
 				(path "/3e989608-eeda-4a48-bc6c-c5e1d1678702/f7bd652a-238e-4a19-a7e7-e5372eb58a34"
-					(reference "C23")
+					(reference "C22")
 					(unit 1)
 				)
@@
 		(in_pos_files yes)
 		(dnp no)
-		(property "Reference" "#PWR038"
+		(property "Reference" "#PWR037"
 			(at 50.8 64.77 0)
 			(hide yes)
@@
 			(project "demo LoRa_Node"
 				(path "/3e989608-eeda-4a48-bc6c-c5e1d1678702/f7bd652a-238e-4a19-a7e7-e5372eb58a34"
-					(reference "#PWR038")
+					(reference "#PWR037")
 					(unit 1)
 				)
@@
 		(in_pos_files yes)
 		(dnp no)
-		(property "Reference" "C28"
+		(property "Reference" "C27"
 			(at 236.22 96.52 0)
 			(show_name no)
@@
 			(project "demo LoRa_Node"
 				(path "/3e989608-eeda-4a48-bc6c-c5e1d1678702/f7bd652a-238e-4a19-a7e7-e5372eb58a34"
-					(reference "C28")
+					(reference "C27")
 					(unit 1)
 				)
@@
 		(in_pos_files yes)
 		(dnp no)
-		(property "Reference" "C22"
+		(property "Reference" "C21"
 			(at 82.55 49.53 90)
 			(show_name no)
@@
 			(project "demo LoRa_Node"
 				(path "/3e989608-eeda-4a48-bc6c-c5e1d1678702/f7bd652a-238e-4a19-a7e7-e5372eb58a34"
-					(reference "C22")
+					(reference "C21")
 					(unit 1)
 				)
@@
 		(in_pos_files yes)
 		(dnp no)
-		(property "Reference" "C25"
+		(property "Reference" "C24"
 			(at 125.73 74.93 0)
 			(show_name no)
@@
 			(project "demo LoRa_Node"
 				(path "/3e989608-eeda-4a48-bc6c-c5e1d1678702/f7bd652a-238e-4a19-a7e7-e5372eb58a34"
-					(reference "C25")
+					(reference "C24")
 					(unit 1)
 				)
@@
 		(dnp no)
 		(fields_autoplaced yes)
-		(property "Reference" "#PWR039"
+		(property "Reference" "#PWR038"
 			(at 179.07 77.47 0)
 			(hide yes)
@@
 			(project "demo LoRa_Node"
 				(path "/3e989608-eeda-4a48-bc6c-c5e1d1678702/f7bd652a-238e-4a19-a7e7-e5372eb58a34"
-					(reference "#PWR039")
+					(reference "#PWR038")
 					(unit 1)
 				)
@@
 		(in_pos_files yes)
 		(dnp no)
-		(property "Reference" "#PWR043"
+		(property "Reference" "#PWR042"
 			(at 179.07 113.03 0)
 			(hide yes)
@@
 			(project "demo LoRa_Node"
 				(path "/3e989608-eeda-4a48-bc6c-c5e1d1678702/f7bd652a-238e-4a19-a7e7-e5372eb58a34"
-					(reference "#PWR043")
+					(reference "#PWR042")
 					(unit 1)
 				)
@@
 		(in_pos_files yes)
 		(dnp no)
-		(property "Reference" "#PWR040"
+		(property "Reference" "#PWR039"
 			(at 95.25 90.17 0)
 			(hide yes)
@@
 			(project "demo LoRa_Node"
 				(path "/3e989608-eeda-4a48-bc6c-c5e1d1678702/f7bd652a-238e-4a19-a7e7-e5372eb58a34"
-					(reference "#PWR040")
+					(reference "#PWR039")
 					(unit 1)
 				)
@@
 		(in_pos_files yes)
 		(dnp no)
-		(property "Reference" "#PWR044"
+		(property "Reference" "#PWR043"
 			(at 218.44 113.03 0)
 			(hide yes)
@@
 			(project "demo LoRa_Node"
 				(path "/3e989608-eeda-4a48-bc6c-c5e1d1678702/f7bd652a-238e-4a19-a7e7-e5372eb58a34"
-					(reference "#PWR044")
+					(reference "#PWR043")
 					(unit 1)
 				)
@@
 		(in_pos_files yes)
 		(dnp no)
-		(property "Reference" "C24"
+		(property "Reference" "C23"
 			(at 91.44 74.93 0)
 			(show_name no)
@@
 			(project "demo LoRa_Node"
 				(path "/3e989608-eeda-4a48-bc6c-c5e1d1678702/f7bd652a-238e-4a19-a7e7-e5372eb58a34"
-					(reference "C24")
+					(reference "C23")
 					(unit 1)
 				)
@@
 		(in_pos_files yes)
 		(dnp no)
-		(property "Reference" "C29"
+		(property "Reference" "C28"
 			(at 109.22 106.68 90)
 			(show_name no)
@@
 			(project "demo LoRa_Node"
 				(path "/3e989608-eeda-4a48-bc6c-c5e1d1678702/f7bd652a-238e-4a19-a7e7-e5372eb58a34"
-					(reference "C29")
+					(reference "C28")
 					(unit 1)
 				)
@@
 		(in_pos_files yes)
 		(dnp no)
-		(property "Reference" "#PWR042"
+		(property "Reference" "#PWR041"
 			(at 262.89 101.6 0)
 			(hide yes)
@@
 			(project "demo LoRa_Node"
 				(path "/3e989608-eeda-4a48-bc6c-c5e1d1678702/f7bd652a-238e-4a19-a7e7-e5372eb58a34"
-					(reference "#PWR042")
+					(reference "#PWR041")
 					(unit 1)
 				)
@@
 		(dnp no)
 		(fields_autoplaced yes)
-		(property "Reference" "#PWR037"
+		(property "Reference" "#PWR036"
 			(at 59.69 45.72 0)
 			(hide yes)
@@
 			(project "demo LoRa_Node"
 				(path "/3e989608-eeda-4a48-bc6c-c5e1d1678702/f7bd652a-238e-4a19-a7e7-e5372eb58a34"
-					(reference "#PWR037")
+					(reference "#PWR036")
 					(unit 1)
 				)
@@
 		(in_pos_files yes)
 		(dnp no)
-		(property "Reference" "C30"
+		(property "Reference" "C29"
 			(at 81.28 144.78 0)
 			(show_name no)
@@
 			(project "demo LoRa_Node"
 				(path "/3e989608-eeda-4a48-bc6c-c5e1d1678702/f7bd652a-238e-4a19-a7e7-e5372eb58a34"
-					(reference "C30")
+					(reference "C29")
 					(unit 1)
 				)
@@
 		(in_pos_files yes)
 		(dnp no)
-		(property "Reference" "C27"
+		(property "Reference" "C26"
 			(at 214.63 96.52 0)
 			(show_name no)
@@
 			(project "demo LoRa_Node"
 				(path "/3e989608-eeda-4a48-bc6c-c5e1d1678702/f7bd652a-238e-4a19-a7e7-e5372eb58a34"
-					(reference "C27")
-					(unit 1)
-				)
+					(reference "C26")
+					(unit 1)
+				)
