File: Hardware/Schematics/MCU.kicad_sch (KiCad schematic)
At the start: 31 parts, among them J5 Conn_ARM_SWD_TagConnect_TC2030, SW1 SW_Omron_B3FS, U2 CP2102N-Axx-xQFN28, U3 STM32WL55CCUx, Y1 SG-210STF 32MHz

Commit message: title block update
Other:
- company: (none) -> Nicola Borkowetz
- title: (none) -> LoRa Node MCU

Commit message: adjustment to the power section
Parts:
- renumbered C11 to C10, C12 to C11, C13 to C12, C14 to C13, C7 to C14, C18 to C17, C19 to C18, C20 to C19, C8 to C7, C9 to C8, C10 to C9, R18 to R17
Changed lines of the file:
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@@
 		(in_pos_files yes)
 		(dnp no)
-		(property "Reference" "C9"
+		(property "Reference" "C8"
 			(at 82.55 50.7999 0)
 			(show_name no)
@@
 			(project "demo LoRa_Node"
 				(path "/3e989608-eeda-4a48-bc6c-c5e1d1678702/035a042a-e27c-47a0-bc8b-0546484d86a7"
-					(reference "C9")
+					(reference "C8")
 					(unit 1)
 				)
@@
 		(dnp no)
 		(fields_autoplaced yes)
-		(property "Reference" "#PWR034"
+		(property "Reference" "#PWR033"
 			(at 133.35 165.1 0)
 			(hide yes)
@@
 			(project "demo LoRa_Node"
 				(path "/3e989608-eeda-4a48-bc6c-c5e1d1678702/035a042a-e27c-47a0-bc8b-0546484d86a7"
-					(reference "#PWR034")
+					(reference "#PWR033")
 					(unit 1)
 				)
@@
 		(dnp no)
 		(fields_autoplaced yes)
-		(property "Reference" "#PWR036"
+		(property "Reference" "#PWR035"
 			(at 35.56 191.77 0)
 			(hide yes)
@@
 			(project "demo LoRa_Node"
 				(path "/3e989608-eeda-4a48-bc6c-c5e1d1678702/035a042a-e27c-47a0-bc8b-0546484d86a7"
-					(reference "#PWR036")
+					(reference "#PWR035")
 					(unit 1)
 				)
@@
 		(dnp no)
 		(fields_autoplaced yes)
-		(property "Reference" "#PWR027"
+		(property "Reference" "#PWR026"
 			(at 256.54 93.98 0)
 			(hide yes)
@@
 			(project "demo LoRa_Node"
 				(path "/3e989608-eeda-4a48-bc6c-c5e1d1678702/035a042a-e27c-47a0-bc8b-0546484d86a7"
-					(reference "#PWR027")
+					(reference "#PWR026")
 					(unit 1)
 				)
@@
 		(dnp no)
 		(fields_autoplaced yes)
-		(property "Reference" "C18"
+		(property "Reference" "C17"
 			(at 137.16 170.1799 0)
 			(show_name no)
@@
 			(project "demo LoRa_Node"
 				(path "/3e989608-eeda-4a48-bc6c-c5e1d1678702/035a042a-e27c-47a0-bc8b-0546484d86a7"
-					(reference "C18")
+					(reference "C17")
 					(unit 1)
 				)
@@
 		(in_pos_files yes)
 		(dnp no)
-		(property "Reference" "#PWR031"
+		(property "Reference" "#PWR030"
 			(at 71.12 138.43 0)
 			(hide yes)
@@
 			(project "demo LoRa_Node"
 				(path "/3e989608-eeda-4a48-bc6c-c5e1d1678702/035a042a-e27c-47a0-bc8b-0546484d86a7"
-					(reference "#PWR031")
+					(reference "#PWR030")
 					(unit 1)
 				)
@@
 		(dnp no)
 		(fields_autoplaced yes)
-		(property "Reference" "#PWR028"
+		(property "Reference" "#PWR027"
 			(at 43.18 109.22 0)
 			(hide yes)
@@
 			(project "demo LoRa_Node"
 				(path "/3e989608-eeda-4a48-bc6c-c5e1d1678702/035a042a-e27c-47a0-bc8b-0546484d86a7"
-					(reference "#PWR028")
+					(reference "#PWR027")
 					(unit 1)
 				)
@@
 		(in_pos_files yes)
 		(dnp no)
-		(property "Reference" "C13"
+		(property "Reference" "C12"
 			(at 234.95 107.9499 0)
 			(show_name no)
@@
 			(project "demo LoRa_Node"
 				(path "/3e989608-eeda-4a48-bc6c-c5e1d1678702/035a042a-e27c-47a0-bc8b-0546484d86a7"
-					(reference "C13")
+					(reference "C12")
 					(unit 1)
 				)
@@
 		(dnp no)
 		(fields_autoplaced yes)
-		(property "Reference" "C11"
+		(property "Reference" "C10"
 			(at 163.83 53.3399 0)
 			(show_name no)
@@
 			(project "demo LoRa_Node"
 				(path "/3e989608-eeda-4a48-bc6c-c5e1d1678702/035a042a-e27c-47a0-bc8b-0546484d86a7"
-					(reference "C11")
+					(reference "C10")
 					(unit 1)
 				)
@@
 		(dnp no)
 		(fields_autoplaced yes)
-		(property "Reference" "#FLG03"
+		(property "Reference" "#FLG02"
 			(at 270.51 61.595 0)
 			(hide yes)
@@
 			(project "demo LoRa_Node"
 				(path "/3e989608-eeda-4a48-bc6c-c5e1d1678702/035a042a-e27c-47a0-bc8b-0546484d86a7"
-					(reference "#FLG03")
+					(reference "#FLG02")
 					(unit 1)
 				)
@@
 		(dnp no)
 		(fields_autoplaced yes)
-		(property "Reference" "C19"
+		(property "Reference" "C18"
 			(at 148.59 170.1799 0)
 			(show_name no)
@@
 			(project "demo LoRa_Node"
 				(path "/3e989608-eeda-4a48-bc6c-c5e1d1678702/035a042a-e27c-47a0-bc8b-0546484d86a7"
-					(reference "C19")
+					(reference "C18")
 					(unit 1)
 				)
@@
 		(dnp no)
 		(fields_autoplaced yes)
-		(property "Reference" "#PWR029"
+		(property "Reference" "#PWR028"
 			(at 218.44 127 0)
 			(hide yes)
@@
 			(project "demo LoRa_Node"
 				(path "/3e989608-eeda-4a48-bc6c-c5e1d1678702/035a042a-e27c-47a0-bc8b-0546484d86a7"
-					(reference "#PWR029")
+					(reference "#PWR028")
 					(unit 1)
 				)
@@
 		(dnp no)
 		(fields_autoplaced yes)
-		(property "Reference" "C20"
+		(property "Reference" "C19"
 			(at 160.02 170.1799 0)
 			(show_name no)
@@
 			(project "demo LoRa_Node"
 				(path "/3e989608-eeda-4a48-bc6c-c5e1d1678702/035a042a-e27c-47a0-bc8b-0546484d86a7"
-					(reference "C20")
+					(reference "C19")
 					(unit 1)
 				)
@@
 		(dnp no)
 		(fields_autoplaced yes)
-		(property "Reference" "#PWR035"
+		(property "Reference" "#PWR034"
 			(at 133.35 190.5 0)
 			(hide yes)
@@
 			(project "demo LoRa_Node"
 				(path "/3e989608-eeda-4a48-bc6c-c5e1d1678702/035a042a-e27c-47a0-bc8b-0546484d86a7"
-					(reference "#PWR035")
+					(reference "#PWR034")
 					(unit 1)
 				)
@@
 		(dnp no)
 		(fields_autoplaced yes)
-		(property "Reference" "#FLG05"
+		(property "Reference" "#FLG03"
 			(at 219.71 64.135 0)
 			(hide yes)
@@
 			(project "demo LoRa_Node"
 				(path "/3e989608-eeda-4a48-bc6c-c5e1d1678702/035a042a-e27c-47a0-bc8b-0546484d86a7"
-					(reference "#FLG05")
+					(reference "#FLG03")
 					(unit 1)
 				)
@@
 		(dnp no)
 		(fields_autoplaced yes)
-		(property "Reference" "#PWR030"
+		(property "Reference" "#PWR029"
 			(at 245.11 127 0)
 			(hide yes)
@@
 			(project "demo LoRa_Node"
 				(path "/3e989608-eeda-4a48-bc6c-c5e1d1678702/035a042a-e27c-47a0-bc8b-0546484d86a7"
-					(reference "#PWR030")
+					(reference "#PWR029")
 					(unit 1)
 				)
@@
 		(dnp no)
 		(fields_autoplaced yes)
-		(property "Reference" "C10"
+		(property "Reference" "C9"
 			(at 93.98 50.7999 0)
 			(show_name no)
@@
 			(project "demo LoRa_Node"
 				(path "/3e989608-eeda-4a48-bc6c-c5e1d1678702/035a042a-e27c-47a0-bc8b-0546484d86a7"
-					(reference "C10")
+					(reference "C9")
 					(unit 1)
 				)
@@
 		(dnp no)
 		(fields_autoplaced yes)
-		(property "Reference" "C8"
+		(property "Reference" "C7"
 			(at 35.56 50.7999 0)
 			(show_name no)
@@
 			(project "demo LoRa_Node"
 				(path "/3e989608-eeda-4a48-bc6c-c5e1d1678702/035a042a-e27c-47a0-bc8b-0546484d86a7"
-					(reference "C8")
+					(reference "C7")
 					(unit 1)
 				)
@@
 		(dnp no)
 		(fields_autoplaced yes)
-		(property "Reference" "C7"
+		(property "Reference" "C14"
 			(at 101.6 170.1799 0)
 			(show_name no)
@@
 			(project "demo LoRa_Node"
 				(path "/3e989608-eeda-4a48-bc6c-c5e1d1678702/035a042a-e27c-47a0-bc8b-0546484d86a7"
-					(reference "C7")
+					(reference "C14")
 					(unit 1)
 				)
@@
 		(in_pos_files yes)
 		(dnp no)
-		(property "Reference" "C14"
+		(property "Reference" "C13"
 			(at 248.92 107.9499 0)
 			(show_name no)
@@
 			(project "demo LoRa_Node"
 				(path "/3e989608-eeda-4a48-bc6c-c5e1d1678702/035a042a-e27c-47a0-bc8b-0546484d86a7"
-					(reference "C14")
+					(reference "C13")
 					(unit 1)
 				)
@@
 		(dnp no)
 		(fields_autoplaced yes)
-		(property "Reference" "#FLG02"
+		(property "Reference" "#FLG01"
 			(at 147.32 37.465 0)
 			(hide yes)
@@
 			(project "demo LoRa_Node"
 				(path "/3e989608-eeda-4a48-bc6c-c5e1d1678702/035a042a-e27c-47a0-bc8b-0546484d86a7"
-					(reference "#FLG02")
+					(reference "#FLG01")
 					(unit 1)
 				)
@@
 		(dnp no)
 		(fields_autoplaced yes)
-		(property "Reference" "R18"
+		(property "Reference" "R17"
 			(at 220.98 111.7599 0)
 			(show_name no)
@@
 			(project "demo LoRa_Node"
 				(path "/3e989608-eeda-4a48-bc6c-c5e1d1678702/035a042a-e27c-47a0-bc8b-0546484d86a7"
-					(reference "R18")
+					(reference "R17")
 					(unit 1)
 				)
@@
 		(dnp no)
 		(fields_autoplaced yes)
-		(property "Reference" "#PWR033"
+		(property "Reference" "#PWR032"
 			(at 35.56 163.83 0)
 			(hide yes)
@@
 			(project "demo LoRa_Node"
 				(path "/3e989608-eeda-4a48-bc6c-c5e1d1678702/035a042a-e27c-47a0-bc8b-0546484d86a7"
-					(reference "#PWR033")
+					(reference "#PWR032")
 					(unit 1)
 				)
@@
 		(dnp no)
 		(fields_autoplaced yes)
-		(property "Reference" "#PWR032"
+		(property "Reference" "#PWR031"
 			(at 187.96 146.05 0)
 			(hide yes)
@@
 			(project "demo LoRa_Node"
 				(path "/3e989608-eeda-4a48-bc6c-c5e1d1678702/035a042a-e27c-47a0-bc8b-0546484d86a7"
-					(reference "#PWR032")
+					(reference "#PWR031")
 					(unit 1)
 				)
@@
 		(dnp no)
 		(fields_autoplaced yes)
-		(property "Reference" "C12"
+		(property "Reference" "C11"
 			(at 274.32 72.3899 0)
 			(show_name no)
@@
 			(project "demo LoRa_Node"
 				(path "/3e989608-eeda-4a48-bc6c-c5e1d1678702/035a042a-e27c-47a0-bc8b-0546484d86a7"
-					(reference "C12")
+					(reference "C11")
 					(unit 1)
 				)

Commit message: final hardware V1
Parts:
- R12: value 22k1 -> 46k4
- R16: value 48k7 -> 100k
- R17: value 10k -> 100k
Other:
- moved on the sheet: C10, C11, C12, C13, C5, C6, C7, FB2, FB3, L1, R12, R16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
