File: Hardware/Schematics/analog.kicad_sch (KiCad schematic)
At the start: 27 parts, among them J1 Screw_Terminal_01x04, J2 Screw_Terminal_01x03, J3 Screw_Terminal_01x03, J4 Screw_Terminal_01x03, U1 THVD1400D

Commit message: title block update
Other:
- company: (none) -> Nicola Borkowetz
- title: (none) -> LoRa Node Analog Interface
Changed lines of the file:
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@@
 	(generator_version "10.0")
 	(paper "A4")
+	(title_block
+		(title "LoRa Node Analog Interface")
+		(date "2025-11-28")
+		(rev "A")
+		(company "Nicola Borkowetz")
+	)
 	(junction
 		(at 85.09 88.9)
@@
 		)
 		(instances
-			(project "demo wateranalyser"
+			(project "demo LoRa_Node"
 				(path "/3e989608-eeda-4a48-bc6c-c5e1d1678702/0344d43c-f7c9-496f-9384-ab56684cdcfd"
 					(reference "J3")
@@
 		)
 		(instances
-			(project "demo wateranalyser"
+			(project "demo LoRa_Node"
 				(path "/3e989608-eeda-4a48-bc6c-c5e1d1678702/0344d43c-f7c9-496f-9384-ab56684cdcfd"
 					(reference "C1")
@@
 		)
 		(instances
-			(project "demo wateranalyser"
+			(project "demo LoRa_Node"
 				(path "/3e989608-eeda-4a48-bc6c-c5e1d1678702/0344d43c-f7c9-496f-9384-ab56684cdcfd"
 					(reference "#PWR010")
@@
 		)
 		(instances
-			(project "demo wateranalyser"
+			(project "demo LoRa_Node"
 				(path "/3e989608-eeda-4a48-bc6c-c5e1d1678702/0344d43c-f7c9-496f-9384-ab56684cdcfd"
 					(reference "U1")
@@
 		)
 		(instances
-			(project "demo wateranalyser"
+			(project "demo LoRa_Node"
 				(path "/3e989608-eeda-4a48-bc6c-c5e1d1678702/0344d43c-f7c9-496f-9384-ab56684cdcfd"
 					(reference "J4")
@@
 		)
 		(instances
-			(project "demo wateranalyser"
+			(project "demo LoRa_Node"
 				(path "/3e989608-eeda-4a48-bc6c-c5e1d1678702/0344d43c-f7c9-496f-9384-ab56684cdcfd"
 					(reference "#PWR03")
@@
 		)
 		(instances
-			(project "demo wateranalyser"
+			(project "demo LoRa_Node"
 				(path "/3e989608-eeda-4a48-bc6c-c5e1d1678702/0344d43c-f7c9-496f-9384-ab56684cdcfd"
 					(reference "#PWR08")
@@
 		)
 		(instances
-			(project "demo wateranalyser"
+			(project "demo LoRa_Node"
 				(path "/3e989608-eeda-4a48-bc6c-c5e1d1678702/0344d43c-f7c9-496f-9384-ab56684cdcfd"
 					(reference "#PWR012")
@@
 		)
 		(instances
-			(project "demo wateranalyser"
+			(project "demo LoRa_Node"
 				(path "/3e989608-eeda-4a48-bc6c-c5e1d1678702/0344d43c-f7c9-496f-9384-ab56684cdcfd"
 					(reference "#PWR04")
@@
 		)
 		(instances
-			(project "demo wateranalyser"
+			(project "demo LoRa_Node"
 				(path "/3e989608-eeda-4a48-bc6c-c5e1d1678702/0344d43c-f7c9-496f-9384-ab56684cdcfd"
 					(reference "#PWR011")
@@
 		)
 		(instances
-			(project "demo wateranalyser"
+			(project "demo LoRa_Node"
 				(path "/3e989608-eeda-4a48-bc6c-c5e1d1678702/0344d43c-f7c9-496f-9384-ab56684cdcfd"
 					(reference "J1")
@@
 		)
 		(instances
-			(project "demo wateranalyser"
+			(project "demo LoRa_Node"
 				(path "/3e989608-eeda-4a48-bc6c-c5e1d1678702/0344d43c-f7c9-496f-9384-ab56684cdcfd"
 					(reference "D4")
@@
 		)
 		(instances
-			(project "demo wateranalyser"
+			(project "demo LoRa_Node"
 				(path "/3e989608-eeda-4a48-bc6c-c5e1d1678702/0344d43c-f7c9-496f-9384-ab56684cdcfd"
 					(reference "R6")
@@
 		)
 		(instances
-			(project "demo wateranalyser"
+			(project "demo LoRa_Node"
 				(path "/3e989608-eeda-4a48-bc6c-c5e1d1678702/0344d43c-f7c9-496f-9384-ab56684cdcfd"
 					(reference "#PWR013")
@@
 		)
 		(instances
-			(project "demo wateranalyser"
+			(project "demo LoRa_Node"
 				(path "/3e989608-eeda-4a48-bc6c-c5e1d1678702/0344d43c-f7c9-496f-9384-ab56684cdcfd"
 					(reference "J2")
@@
 		)
 		(instances
-			(project "demo wateranalyser"
+			(project "demo LoRa_Node"
 				(path "/3e989608-eeda-4a48-bc6c-c5e1d1678702/0344d43c-f7c9-496f-9384-ab56684cdcfd"
 					(reference "C3")
@@
 		)
 		(instances
-			(project "demo wateranalyser"
+			(project "demo LoRa_Node"
 				(path "/3e989608-eeda-4a48-bc6c-c5e1d1678702/0344d43c-f7c9-496f-9384-ab56684cdcfd"
 					(reference "D3")
@@
 		)
 		(instances
-			(project "demo wateranalyser"
+			(project "demo LoRa_Node"
 				(path "/3e989608-eeda-4a48-bc6c-c5e1d1678702/0344d43c-f7c9-496f-9384-ab56684cdcfd"
 					(reference "FB1")
@@
 		)
 		(instances
-			(project "demo wateranalyser"
+			(project "demo LoRa_Node"
 				(path "/3e989608-eeda-4a48-bc6c-c5e1d1678702/0344d43c-f7c9-496f-9384-ab56684cdcfd"
 					(reference "R8")
@@
 		)
 		(instances
-			(project "demo wateranalyser"
+			(project "demo LoRa_Node"
 				(path "/3e989608-eeda-4a48-bc6c-c5e1d1678702/0344d43c-f7c9-496f-9384-ab56684cdcfd"
 					(reference "D5")
@@
 		)
 		(instances
-			(project "demo wateranalyser"
+			(project "demo LoRa_Node"
 				(path "/3e989608-eeda-4a48-bc6c-c5e1d1678702/0344d43c-f7c9-496f-9384-ab56684cdcfd"
 					(reference "R1")
@@
 		)
 		(instances
-			(project "demo wateranalyser"
+			(project "demo LoRa_Node"
 				(path "/3e989608-eeda-4a48-bc6c-c5e1d1678702/0344d43c-f7c9-496f-9384-ab56684cdcfd"
 					(reference "#PWR01")
@@
 		)
 		(instances
-			(project "demo wateranalyser"
+			(project "demo LoRa_Node"
 				(path "/3e989608-eeda-4a48-bc6c-c5e1d1678702/0344d43c-f7c9-496f-9384-ab56684cdcfd"
 					(reference "R9")
@@
 		)
 		(instances
-			(project "demo wateranalyser"
+			(project "demo LoRa_Node"
 				(path "/3e989608-eeda-4a48-bc6c-c5e1d1678702/0344d43c-f7c9-496f-9384-ab56684cdcfd"
 					(reference "R10")
@@
 		)
 		(instances
-			(project "demo wateranalyser"
+			(project "demo LoRa_Node"
 				(path "/3e989608-eeda-4a48-bc6c-c5e1d1678702/0344d43c-f7c9-496f-9384-ab56684cdcfd"
 					(reference "D1")
@@
 		)
 		(instances
-			(project "demo wateranalyser"
+			(project "demo LoRa_Node"
 				(path "/3e989608-eeda-4a48-bc6c-c5e1d1678702/0344d43c-f7c9-496f-9384-ab56684cdcfd"
 					(reference "F1")
@@
 		)
 		(instances
-			(project "demo wateranalyser"
+			(project "demo LoRa_Node"
 				(path "/3e989608-eeda-4a48-bc6c-c5e1d1678702/0344d43c-f7c9-496f-9384-ab56684cdcfd"
 					(reference "R11")
@@
 		)
 		(instances
-			(project "demo wateranalyser"
+			(project "demo LoRa_Node"
 				(path "/3e989608-eeda-4a48-bc6c-c5e1d1678702/0344d43c-f7c9-496f-9384-ab56684cdcfd"
 					(reference "C2")
@@
 		)
 		(instances
-			(project "demo wateranalyser"
+			(project "demo LoRa_Node"
 				(path "/3e989608-eeda-4a48-bc6c-c5e1d1678702/0344d43c-f7c9-496f-9384-ab56684cdcfd"
 					(reference "#PWR07")
@@
 		)
 		(instances
-			(project "demo wateranalyser"
+			(project "demo LoRa_Node"
 				(path "/3e989608-eeda-4a48-bc6c-c5e1d1678702/0344d43c-f7c9-496f-9384-ab56684cdcfd"
 					(reference "C4")
@@
 		)
 		(instances
-			(project "demo wateranalyser"
+			(project "demo LoRa_Node"
 				(path "/3e989608-eeda-4a48-bc6c-c5e1d1678702/0344d43c-f7c9-496f-9384-ab56684cdcfd"
 					(reference "R7")
@@
 		)
 		(instances
-			(project "demo wateranalyser"
+			(project "demo LoRa_Node"
 				(path "/3e989608-eeda-4a48-bc6c-c5e1d1678702/0344d43c-f7c9-496f-9384-ab56684cdcfd"
 					(reference "#PWR02")
@@
 		)
 		(instances
-			(project "demo wateranalyser"
+			(project "demo LoRa_Node"
 				(path "/3e989608-eeda-4a48-bc6c-c5e1d1678702/0344d43c-f7c9-496f-9384-ab56684cdcfd"
 					(reference "#PWR014")
@@
 		)
 		(instances
-			(project "demo wateranalyser"
+			(project "demo LoRa_Node"
 				(path "/3e989608-eeda-4a48-bc6c-c5e1d1678702/0344d43c-f7c9-496f-9384-ab56684cdcfd"
 					(reference "R4")
@@
 		)
 		(instances
-			(project "demo wateranalyser"
+			(project "demo LoRa_Node"
 				(path "/3e989608-eeda-4a48-bc6c-c5e1d1678702/0344d43c-f7c9-496f-9384-ab56684cdcfd"
 					(reference "R5")
@@
 		)
 		(instances
-			(project "demo wateranalyser"
+			(project "demo LoRa_Node"
 				(path "/3e989608-eeda-4a48-bc6c-c5e1d1678702/0344d43c-f7c9-496f-9384-ab56684cdcfd"
 					(reference "#PWR09")
@@
 		)
 		(instances
-			(project "demo wateranalyser"
+			(project "demo LoRa_Node"
 				(path "/3e989608-eeda-4a48-bc6c-c5e1d1678702/0344d43c-f7c9-496f-9384-ab56684cdcfd"
 					(reference "R3")
@@
 		)
 		(instances
-			(project "demo wateranalyser"
+			(project "demo LoRa_Node"
 				(path "/3e989608-eeda-4a48-bc6c-c5e1d1678702/0344d43c-f7c9-496f-9384-ab56684cdcfd"
 					(reference "D2")
@@
 		)
 		(instances
-			(project "demo wateranalyser"
+			(project "demo LoRa_Node"
 				(path "/3e989608-eeda-4a48-bc6c-c5e1d1678702/0344d43c-f7c9-496f-9384-ab56684cdcfd"
 					(reference "R2")
@@
 		)
 		(instances
-			(project "demo wateranalyser"
+			(project "demo LoRa_Node"
 				(path "/3e989608-eeda-4a48-bc6c-c5e1d1678702/0344d43c-f7c9-496f-9384-ab56684cdcfd"
 					(reference "#PWR05")
@@
 		)
 		(instances
-			(project "demo wateranalyser"
+			(project "demo LoRa_Node"
 				(path "/3e989608-eeda-4a48-bc6c-c5e1d1678702/0344d43c-f7c9-496f-9384-ab56684cdcfd"
 					(reference "#PWR06")

Commit message: final hardware V1
Other:
- moved on the sheet: C1
Changed lines of the file:
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@@
 	)
 	(junction
-		(at 186.69 43.18)
-		(diameter 0)
-		(color 0 0 0 0)
-	)
-	(junction
 		(at 63.5 91.44)
 		(diameter 0)
@@
 	)
 	(junction
+		(at 186.69 43.18)
+		(diameter 0)
+		(color 0 0 0 0)
+	)
+	(junction
 		(at 104.14 177.8)
 		(diameter 0)
@@
 	)
 	(junction
+		(at 186.69 31.75)
+		(diameter 0)
+		(color 0 0 0 0)
+	)
+	(junction
 		(at 81.28 59.69)
 		(diameter 0)
@@
 	(wire
 		(pts
-			(xy 227.33 30.48) (xy 227.33 34.29)
-		)
-		(stroke
-			(width 0)
-			(type default)
-		)
-	)
-	(wire
-		(pts
 			(xy 49.53 88.9) (xy 85.09 88.9)
 		)
@@
 	(wire
 		(pts
-			(xy 63.5 91.44) (xy 91.44 91.44)
+			(xy 186.69 25.4) (xy 186.69 31.75)
 		)
 		(stroke
@@
 	(wire
 		(pts
-			(xy 49.53 165.1) (xy 54.61 165.1)
+			(xy 63.5 91.44) (xy 91.44 91.44)
 		)
 		(stroke
@@
 	(wire
 		(pts
-			(xy 186.69 36.83) (xy 186.69 43.18)
+			(xy 49.53 165.1) (xy 54.61 165.1)
 		)
 		(stroke
@@
 	(wire
 		(pts
+			(xy 186.69 31.75) (xy 186.69 43.18)
+		)
+		(stroke
+			(width 0)
+			(type default)
+		)
+	)
+	(wire
+		(pts
 			(xy 104.14 91.44) (xy 104.14 96.52)
 		)
@@
 	(wire
 		(pts
+			(xy 171.45 31.75) (xy 171.45 34.29)
+		)
+		(stroke
+			(width 0)
+			(type default)
+		)
+	)
+	(wire
+		(pts
 			(xy 143.51 62.23) (xy 168.91 62.23)
 		)
@@
 	(wire
 		(pts
-			(xy 227.33 41.91) (xy 227.33 44.45)
+			(xy 171.45 31.75) (xy 186.69 31.75)
+		)
+		(stroke
+			(width 0)
+			(type default)
+		)
+	)
+	(wire
+		(pts
+			(xy 171.45 41.91) (xy 171.45 44.45)
 		)
 		(stroke
@@
 	(symbol
 		(lib_id "Device:C")
-		(at 227.33 38.1 0)
+		(at 171.45 38.1 0)
 		(unit 1)
 		(body_style 1)
@@
 		(fields_autoplaced yes)
 		(property "Reference" "C1"
-			(at 231.14 36.8299 0)
+			(at 175.26 36.8299 0)
 			(show_name no)
 			(do_not_autoplace no)
@@
 		)
 		(property "Value" "100n"
-			(at 231.14 39.3699 0)
+			(at 175.26 39.3699 0)
 			(show_name no)
 			(do_not_autoplace no)
@@
 		)
 		(property "Footprint" "Capacitor_SMD:C_0603_1608Metric"
-			(at 228.2952 41.91 0)
+			(at 172.4152 41.91 0)
 			(hide yes)
 			(show_name no)
@@
 		)
 		(property "Datasheet" ""
-			(at 227.33 38.1 0)
+			(at 171.45 38.1 0)
 			(hide yes)
 			(show_name no)
@@
 		)
 		(property "Description" "Unpolarized capacitor"
-			(at 227.33 38.1 0)
+			(at 171.45 38.1 0)
 			(hide yes)
 			(show_name no)
@@
 	)
 	(symbol
-		(lib_id "power:+5V")
-		(at 227.33 30.48 0)
-		(unit 1)
-		(body_style 1)
-		(exclude_from_sim no)
-		(in_bom yes)
-		(on_board yes)
-		(in_pos_files yes)
-		(dnp no)
-		(fields_autoplaced yes)
-		(property "Reference" "#PWR03"
-			(at 227.33 34.29 0)
-			(hide yes)
-			(show_name no)
-			(do_not_autoplace no)
-			(effects
-				(font
-					(size 1.27 1.27)
-				)
-			)
-		)
-		(property "Value" "+3V3"
-			(at 227.33 25.4 0)
-			(show_name no)
-			(do_not_autoplace no)
-			(effects
-				(font
-					(size 1.27 1.27)
-				)
-			)
-		)
-		(property "Footprint" ""
-			(at 227.33 30.48 0)
-			(hide yes)
-			(show_name no)
-			(do_not_autoplace no)
-			(effects
-				(font
-					(size 1.27 1.27)
-				)
-			)
-		)
-		(property "Datasheet" ""
-			(at 227.33 30.48 0)
-			(hide yes)
-			(show_name no)
-			(do_not_autoplace no)
-			(effects
-				(font
-					(size 1.27 1.27)
-				)
-			)
-		)
-		(property "Description" "Power symbol creates a global label with name \"+5V\""
-			(at 227.33 30.48 0)
-			(hide yes)
-			(show_name no)
-			(do_not_autoplace no)
-			(effects
-				(font
-					(size 1.27 1.27)
-				)
-			)
-		)
-		(pin "1"
-		)
-		(instances
-			(project "demo LoRa_Node"
-				(path "/3e989608-eeda-4a48-bc6c-c5e1d1678702/0344d43c-f7c9-496f-9384-ab56684cdcfd"
-					(reference "#PWR03")
-					(unit 1)
-				)
-			)
-		)
-	)
-	(symbol
 		(lib_id "power:GND")
 		(at 186.69 87.63 0)
@@
 	(symbol
 		(lib_id "power:+5V")
-		(at 186.69 36.83 0)
+		(at 186.69 25.4 0)
 		(unit 1)
 		(body_style 1)
@@
 		(in_pos_files yes)
 		(dnp no)
-		(fields_autoplaced yes)
 		(property "Reference" "#PWR04"
-			(at 186.69 40.64 0)
+			(at 186.69 29.21 0)
 			(hide yes)
 			(show_name no)
@@
 		)
 		(property "Value" "+3V3"
-			(at 186.69 31.75 0)
+			(at 186.69 21.082 0)
 			(show_name no)
 			(do_not_autoplace no)
@@
 		)
 		(property "Footprint" ""
-			(at 186.69 36.83 0)
+			(at 186.69 25.4 0)
 			(hide yes)
 			(show_name no)
@@
 		)
 		(property "Datasheet" ""
-			(at 186.69 36.83 0)
+			(at 186.69 25.4 0)
 			(hide yes)
 			(show_name no)
@@
 		)
 		(property "Description" "Power symbol creates a global label with name \"+5V\""
-			(at 186.69 36.83 0)
+			(at 186.69 25.4 0)
 			(hide yes)
 			(show_name no)
@@
 	(symbol
 		(lib_id "power:GND")
-		(at 227.33 44.45 0)
+		(at 171.45 44.45 0)
 		(unit 1)
 		(body_style 1)
@@
 		(fields_autoplaced yes)
 		(property "Reference" "#PWR05"
-			(at 227.33 50.8 0)
+			(at 171.45 50.8 0)
 			(hide yes)
 			(show_name no)
@@
 		)
 		(property "Value" "GND"
-			(at 227.33 49.53 0)
+			(at 171.45 49.53 0)
 			(show_name no)
 			(do_not_autoplace no)
@@
 		)
 		(property "Footprint" ""
-			(at 227.33 44.45 0)
+			(at 171.45 44.45 0)
 			(hide yes)
 			(show_name no)
@@
 		)
 		(property "Datasheet" ""
-			(at 227.33 44.45 0)
+			(at 171.45 44.45 0)
 			(hide yes)
 			(show_name no)
@@
 		)
 		(property "Description" "Power symbol creates a global label with name \"GND\" , ground"
-			(at 227.33 44.45 0)
+			(at 171.45 44.45 0)
 			(hide yes)
 			(show_name no)
